File: mini_cicd_tests/mini_cicd_tests.kicad_pcb (KiCad board)
At the start: 0 parts

Commit message: Add test board
Parts:
- added BT101: Battery_Cell, Battery:Battery_Panasonic_CR2025-V1AK_Vertical_CircularHoles, F.Cu at (123.2, 81.3)
- added D101: LED, LED_SMD:LED_0805_2012Metric_Pad1.15x1.40mm_HandSolder, F.Cu at (130.4, 88.3)
- added R101: 470R, Resistor_SMD:R_0805_2012Metric_Pad1.20x1.40mm_HandSolder, F.Cu at (125.7, 88.3)
Routing:
- net Net-(BT101--): track 0.00 -> 10.9 mm
- net Net-(BT101-+): track 0.00 -> 7.67 mm
- net Net-(D101-A): track 0.00 -> 2.74 mm
Other:
- board outline added: 26.7 x 19.7 mm
- copper layers 0 -> 2
