File: mini_cicd_tests/mini_cicd_tests.kicad_sch (KiCad schematic)
At the start: 3 parts

Commit message: Add test board
Parts:
- BT101: footprint (none) -> Battery:Battery_Panasonic_CR2025-V1AK_Vertical_CircularHoles
- D101: footprint (none) -> LED_SMD:LED_0805_2012Metric_Pad1.15x1.40mm_HandSolder
- R101: value R -> 470R; footprint (none) -> Resistor_SMD:R_0805_2012Metric_Pad1.20x1.40mm_HandSolder
Changed lines of the file:
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@@
 			)
 		)
-		(property "Footprint" ""
+		(property "Footprint" "Battery:Battery_Panasonic_CR2025-V1AK_Vertical_CircularHoles"
 			(at 83.82 81.026 90)
 			(effects
@@
 			)
 		)
-		(property "Value" "R"
+		(property "Value" "470R"
 			(at 105.41 78.7399 0)
 			(effects
@@
 			)
 		)
-		(property "Footprint" ""
+		(property "Footprint" "Resistor_SMD:R_0805_2012Metric_Pad1.20x1.40mm_HandSolder"
 			(at 101.092 77.47 90)
 			(effects
@@
 			)
 		)
-		(property "Footprint" ""
+		(property "Footprint" "LED_SMD:LED_0805_2012Metric_Pad1.15x1.40mm_HandSolder"
 			(at 102.87 88.9 0)
 			(effects
